Commit message: got it working yay

File: src/catbot_pybullet/description/robot.urdf (robot description, URDF)
Before this commit: robot catbot, 11 links, 10 joints
Links:
- added link lower_thigh_lower_thigh, mass 0.135358; collision mesh filename=package://catbot_pybullet/meshes/lower_thigh.stl; visual mesh filename=package://catbot_pybullet/meshes/lower_thigh.stl
- added link lower_to_upper_thigh_connector_d_shaft_lower_motor, mass 0.0183559; collision mesh filename=package://catbot_pybullet/meshes/d_shaft_lower_motor.stl; visual mesh filename=package://catbot_pybullet/meshes/d_shaft_lower_motor.stl
- added link lower_to_upper_thigh_connector_grainger_35jc77_3, mass 1e-09; collision mesh filename=package://catbot_pybullet/meshes/grainger_35jc77.stl; visual mesh filename=package://catbot_pybullet/meshes/grainger_35jc77.stl
- added link lower_to_upper_thigh_connector_lower_to_upper_thigh_connector, mass 0.0185659; collision mesh filename=package://catbot_pybullet/meshes/lower_to_upper_thigh_conne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; visual mesh filename=package://catbot_pybullet/meshes/lower_to_upper_thigh_conne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
- added link lower_to_upper_thigh_connector_pins_3, mass 0.0115862; collision mesh filename=package://catbot_pybullet/meshes/pins.stl; visual mesh filename=package://catbot_pybullet/meshes/pins.stl
- added link part_1_part_1, mass 0.346789; collision mesh filename=package://catbot_pybullet/meshes/part_1.stl; visual mesh filename=package://catbot_pybullet/meshes/part_1.stl
- added link shin_grainger_35jc77_6, mass 1e-09; collision mesh filename=package://catbot_pybullet/meshes/grainger_35jc77.stl; visual mesh filename=package://catbot_pybullet/meshes/grainger_35jc77.stl
- added link shin_grainger_35jc77_7, mass 1e-09; collision mesh filename=package://catbot_pybullet/meshes/grainger_35jc77.stl; visual mesh filename=package://catbot_pybullet/meshes/grainger_35jc77.stl
- added link shin_pins_4, mass 0.0115862; collision mesh filename=package://catbot_pybullet/meshes/pins.stl; visual mesh filename=package://catbot_pybullet/meshes/pins.stl
- added link shin_pins_5, mass 0.0115862; collision mesh filename=package://catbot_pybullet/meshes/pins.stl; visual mesh filename=package://catbot_pybullet/meshes/pins.stl
- added link shin_shin, mass 0.049659; collision mesh filename=package://catbot_pybullet/meshes/shin.stl; visual mesh filename=package://catbot_pybullet/meshes/shin.stl
- added link upper_link_1_d_shaft_upper_motor, mass 0.0169769; collision mesh filename=package://catbot_pybullet/meshes/d_shaft_upper_motor.stl; visual mesh filename=package://catbot_pybullet/meshes/d_shaft_upper_motor.stl
- added link upper_link_1_upper_link_1, mass 0.051287; collision mesh filename=package://catbot_pybullet/meshes/upper_link_1.stl; visual mesh filename=package://catbot_pybullet/meshes/upper_link_1.stl
- added link upper_link_2_grainger_35jc77, mass 1e-09; collision mesh filename=package://catbot_pybullet/meshes/grainger_35jc77.stl; visual mesh filename=package://catbot_pybullet/meshes/grainger_35jc77.stl
- added link upper_link_2_grainger_35jc77_2, mass 1e-09; collision mesh filename=package://catbot_pybullet/meshes/grainger_35jc77.stl; visual mesh filename=package://catbot_pybullet/meshes/grainger_35jc77.stl
- added link upper_link_2_pins, mass 0.0115862; collision mesh filename=package://catbot_pybullet/meshes/pins.stl; visual mesh filename=package://catbot_pybullet/meshes/pins.stl
- added link upper_link_2_pins_2, mass 0.0115862; collision mesh filename=package://catbot_pybullet/meshes/pins.stl; visual mesh filename=package://catbot_pybullet/meshes/pins.stl
- added link upper_link_2_upper_link_2, mass 0.0328541; collision mesh filename=package://catbot_pybullet/meshes/upper_link_2.stl; visual mesh filename=package://catbot_pybullet/meshes/upper_link_2.stl
- added link upper_thigh_grainger_35jc77_4, mass 1e-09; collision mesh filename=package://catbot_pybullet/meshes/grainger_35jc77.stl; visual mesh filename=package://catbot_pybullet/meshes/grainger_35jc77.stl
- added link upper_thigh_grainger_35jc77_5, mass 1e-09; collision mesh filename=package://catbot_pybullet/meshes/grainger_35jc77.stl; visual mesh filename=package://catbot_pybullet/meshes/grainger_35jc77.stl
- added link upper_thigh_upper_thigh, mass 0.139251; collision mesh filename=package://catbot_pybullet/meshes/upper_thigh.stl; visual mesh filename=package://catbot_pybullet/meshes/upper_thigh.stl
- link lower_thigh: geometry 
- link lower_to_upper_thigh_connector: mass 0.0299421 -> 1e-09; geometry 
- link part_1: geometry 
- link shin: mass 0.0231725 -> 1e-09; geometry 
- link upper_link_1: geometry 
- link upper_link_2: mass 0.0231725 -> 1e-09; geometry 
- link upper_thigh: geometry 
Joints:
- added joint lower_thigh_lower_thigh_fixed: type fixed, parent lower_thigh, child lower_thigh_lower_thigh, origin xyz=9.61386e-05 -0.1125 0.0001 rpy=-1.5708 1.26729e-15 -1.56994, axis 0 0 1, limit effort=10 velocity=10
- added joint lower_to_upper_thigh_connector_d_shaft_lower_motor_fixed: type fixed, parent lower_to_upper_thigh_connector, child lower_to_upper_thigh_connector_d_shaft_lower_motor, origin xyz=0 0 0.0334109 rpy=5.77848e-17 -4.93476e-16 0, axis 0 0 1, limit effort=10 velocity=10
- added joint lower_to_upper_thigh_connector_grainger_35jc77_3_fixed: type fixed, parent lower_to_upper_thigh_connector, child lower_to_upper_thigh_connector_grainger_35jc77_3, origin xyz=-0.000995748 -0.060184 0.0224252 rpy=-8.20465e-16 5.49234e-16 3.12684, axis 0 0 1, limit effort=10 velocity=10
- added joint lower_to_upper_thigh_connector_lower_to_upper_thigh_connector_fixed: type fixed, parent lower_to_upper_thigh_connector, child lower_to_upper_thigh_connector_lower_to_upper_thigh_connector, origin xyz=-0.000553083 -0.0301873 0.0259964 rpy=1.5708 -8.58882e-16 1.55604, axis 0 0 1, limit effort=10 velocity=10
- added joint lower_to_upper_thigh_connector_pins_3_fixed: type fixed, parent lower_to_upper_thigh_connector, child lower_to_upper_thigh_connector_pins_3, origin xyz=-0.000995748 -0.060184 0.0329252 rpy=1.5708 -6.63175e-16 1.55604, axis 0 0 1, limit effort=10 velocity=10
- added joint part_1_part_1_fixed: type fixed, parent part_1, child part_1_part_1, origin xyz=0.0907012 0.0564074 0.263581 rpy=-1.5708 -4.85085e-10 -3.14159, axis 0 0 1, limit effort=10 velocity=10
- added joint shin_grainger_35jc77_6_fixed: type fixed, parent shin, child shin_grainger_35jc77_6, origin xyz=-0.06 -7.63278e-17 -0.0091 rpy=-3.1225e-16 7.97973e-17 3.14159, axis 0 0 1, limit effort=10 velocity=10
- added joint shin_grainger_35jc77_7_fixed: type fixed, parent shin, child shin_grainger_35jc77_7, origin xyz=0 0 -0.0091 rpy=-2.01228e-16 1.04083e-16 -3.14159, axis 0 0 1, limit effort=10 velocity=10
- added joint shin_pins_4_fixed: type fixed, parent shin, child shin_pins_4, origin xyz=-0.06 -7.63278e-17 0.0014 rpy=1.5708 3.1225e-16 -1.5708, axis 0 0 1, limit effort=10 velocity=10
- added joint shin_pins_5_fixed: type fixed, parent shin, child shin_pins_5, origin xyz=0 0 0.0014 rpy=1.5708 -4.93038e-32 0, axis 0 0 1, limit effort=10 velocity=10
- added joint shin_shin_fixed: type fixed, parent shin, child shin_shin, origin xyz=-0.08 -4.16334e-17 -0.0126712 rpy=-1.5708 1.37732e-16 -3.14159, axis 0 0 1, limit effort=10 velocity=10
- added joint upper_link_1_d_shaft_upper_motor_fixed: type fixed, parent upper_link_1, child upper_link_1_d_shaft_upper_motor, origin xyz=0 0 0.0117 rpy=-1.5708 -0 0, axis 0 0 1, limit effort=10 velocity=10
- added joint upper_link_1_upper_link_1_fixed: type fixed, parent upper_link_1, child upper_link_1_upper_link_1, origin xyz=8.32667e-17 -0.04 0.0297 rpy=1.5708 5.13253e-17 1.5708, axis 0 0 1, limit effort=10 velocity=10
- added joint upper_link_2_grainger_35jc77_2_fixed: type fixed, parent upper_link_2, child upper_link_2_grainger_35jc77_2, origin xyz=-6.64399e-16 -0.105 -0.0091 rpy=-7.17371e-18 -9.17139e-17 -3.88578e-16, axis 0 0 1, limit effort=10 velocity=10
- added joint upper_link_2_grainger_35jc77_fixed: type fixed, parent upper_link_2, child upper_link_2_grainger_35jc77, origin xyz=-1.21431e-17 0 -0.0091 rpy=8.30319e-17 -1.29878e-16 2.22045e-16, axis 0 0 1, limit effort=10 velocity=10
- added joint upper_link_2_pins_2_fixed: type fixed, parent upper_link_2, child upper_link_2_pins_2, origin xyz=-1.21431e-17 0 -0.0196 rpy=-1.5708 3.69779e-32 -5.55112e-17, axis 0 0 1, limit effort=10 velocity=10
- added joint upper_link_2_pins_fixed: type fixed, parent upper_link_2, child upper_link_2_pins, origin xyz=-6.64399e-16 -0.105 0.0014 rpy=1.5708 2.9476e-17 -1.5708, axis 0 0 1, limit effort=10 velocity=10
- added joint upper_link_2_upper_link_2_fixed: type fixed, parent upper_link_2, child upper_link_2_upper_link_2, origin xyz=-3.17454e-16 -0.0525 -0.00552876 rpy=1.5708 -1.5289e-16 -1.5708, axis 0 0 1, limit effort=10 velocity=10
- added joint upper_thigh_grainger_35jc77_4_fixed: type fixed, parent upper_thigh, child upper_thigh_grainger_35jc77_4, origin xyz=5.55112e-17 2.77556e-17 -0.0247928 rpy=-3.14159 2.72047e-16 0.014756, axis 0 0 1, limit effort=10 velocity=10
- added joint upper_thigh_grainger_35jc77_5_fixed: type fixed, parent upper_thigh, child upper_thigh_grainger_35jc77_5, origin xyz=5.55112e-17 2.77556e-17 -0.00950784 rpy=-3.14159 4.11437e-16 -1.55604, axis 0 0 1, limit effort=10 velocity=10
- added joint upper_thigh_upper_thigh_fixed: type fixed, parent upper_thigh, child upper_thigh_upper_thigh, origin xyz=5.55112e-17 2.77556e-17 -0.0261503 rpy=-1.5708 2.72047e-16 0.014756, axis 0 0 1, limit effort=10 velocity=10
- joint closing_passive3_1_frame: origin xyz=-0.06 6.245e-17 -7.32785e-17 rpy=-1.66533e-16 2.56739e-16 -1.5708 -> xyz=-0.06 -7.63278e-17 -1.14478e-16 rpy=1.07493e-16 3.1225e-16 -1.5708
- joint closing_passive3_2_frame: origin xyz=0.149272 -0.168354 7.34682e-17 rpy=3.14159 3.26486e-16 2.29619 -> xyz=0.000192277 -0.225 -2.24091e-16 rpy=3.14159 -1.26729e-15 1.57165
- joint closing_passive5_1_frame: origin xyz=-3.33067e-16 -0.105 2.47008e-16 rpy=1.7087e-16 3.1225e-16 -1.5708 -> xyz=-6.64399e-16 -0.105 3.52948e-16 rpy=2.02456e-16 2.9476e-17 -1.5708
- joint closing_passive5_2_frame: origin xyz=-0.133045 -0.12124 -0.0262503 rpy=3.14159 -1.62533e-16 2.30981 -> xyz=-0.17998 -0.00265599 -0.0262503 rpy=-3.14159 -8.56631e-16 1.58555
- joint motor1: child part_1 -> upper_link_1; limit effort=50 velocity=50 -> lower=-0.780544 upper=1.96935 effort=50 velocity=50; origin xyz=-0.0728365 0.0296822 0.227745 rpy=-1.5708 1.05526 -3.14159 -> xyz=-0.0728365 0.0296822 0.227745 rpy=1.5708 1.5708 0; parent upper_link_1 -> part_1; type passive -> revolute
- joint motor2: limit effort=50 velocity=50 -> lower=-3.141592653589793 upper=3.141592653589793 effort=50 velocity=50; origin xyz=-0.0638436 0.112669 -0.00172517 rpy=3.14159 -3.65185e-16 -3.11074 -> xyz=0.0566635 0.0314074 0.227745 rpy=1.5708 -0.539689 -4.21394e-16; type passive -> revolute
- joint passive1: origin xyz=-0.000995748 0.060184 -0.0315252 rpy=-4.58531e-16 8.32885e-16 -1.55604 -> xyz=-0.000995748 -0.060184 0.0315252 rpy=3.14159 -6.63175e-16 1.55604; type passive -> continuous
- joint passive2: origin xyz=-0.166306 -0.15155 -0.0262503 rpy=3.14159 -4.52115e-17 -1.55708 -> xyz=-0.224976 -0.00331998 -0.0262503 rpy=-3.14159 2.5947e-16 -1.55425; type passive -> continuous
- joint passive4: limit effort=10 velocity=10 -> lower=-0.958899 upper=0.958899 effort=10 velocity=10; origin xyz=2.77556e-17 1.38778e-17 -0.00527485 rpy=0 -1.47911e-31 5.55112e-17 -> xyz=0 0 0.00527485 rpy=3.14159 1.72563e-31 0; type passive -> revolute
- joint passive6: origin xyz=-0.142439 -0.000117766 0.267185 rpy=1.5708 -0.288133 4.01667e-16 -> xyz=8.32667e-17 -0.08 0.0298 rpy=8.7803e-17 1.71793e-16 2.10804; type passive -> continuous

Commit message: yay

File: src/catbot_pybullet/description/robot.urdf (robot description, URDF)
Before this commit: robot catbot, 32 links, 31 joints
Links:
- link part_1: mass 0 -> 1e-09

Commit message: jump works now yay

File: src/catbot_pybullet/description/robot.urdf (robot description, URDF)
Before this commit: robot catbot, 32 links, 31 joints
Links:
- link part_1_part_1: mass 0.346789 -> 3.46789
